File: kicad/DAC.sch (KiCad schematic (older format))
At the start: 0 parts

Commit message: move DAC circuit to sheet
Parts:
- added C? (x11): 0.1uF, Capacitor_SMD:C_0805_2012Metric, symbol Device:C_Small
- added C?: 1uF, Capacitor_SMD:C_0805_2012Metric_Pad1.15x1.40mm_HandSolder, symbol Device:C
- added C?: 1uF, Capacitor_SMD:C_0805_2012Metric, symbol Device:C_Small
- added Q? (x2): Q_DUAL_NMOS_S1G1D2S2G2D1, symbol Device:Q_DUAL_NMOS_S1G1D2S2G2D1
- added R? (x8): 1k, Resistor_SMD:R_0805_2012Metric, symbol Device:R
- added R? (x2): 4.7k, Resistor_SMD:R_0805_2012Metric_Pad1.15x1.40mm_HandSolder, symbol Device:R
- added U?: DS3911, quadrant:SON40P300X500X80-15N, symbol quadrant:DS3911
- added U? (x5): TSV994IPT, Package_SO:TSSOP-14_4.4x5mm_P0.65mm, symbol Device:Opamp_Quad_Generic
- added U?: TCR2EE48, Package_TO_SOT_SMD:SOT-553, symbol quadrant:TCR2EE
Connections:
- new net: R?.1, U?.1 (DAC0)
- new net: R?.1, U?.2 (DAC1)
- new net: R?.1, U?.5 (DAC2)
- new net: R?.1, U?.6 (DAC3)
- new net: C?.2, R?.1, R?.2 (x4)
- new net: C?.2, R?.2, U?.3 (+)
- new net: C?.2, R?.2, U?.5 (+)
- new net: C?.2, R?.2, U?.10 (+)
- new net: C?.2, R?.2, U?.12 (+)
- new net: C?.2, U?.11 (V-)
- new net: C?.1, U?.4 (V+)
- new net +3V3: Q?.2 (G), Q?.5 (G)
- new net 4v8: C?.1, C?.1, U?.3 (VREF), U?.4 (VOUT)
- new net DAC0: U?.1, U?.2 (-)
- new net DAC1: U?.6 (-), U?.7
- new net DAC2: U?.8, U?.9 (-)
- new net DAC3: U?.13 (-), U?.14
- new net GND: C?.1, C?.1, C?.1, C?.1, C?.1, C?.1, C?.1, C?.1, C?.1, C?.1, C?.2, C?.2, C?.2, C?.2, R?.1, R?.1, U?.1 (CTRL), U?.10 (A1), U?.11 (A0), U?.14 (VCC), U?.15 (Epad), U?.2 (GND), U?.3 (VIN), U?.4 (GND), U?.9 (GND)
- new net SCL: Q?.4 (S), R?.2, U?.13 (SCL)
- new net SCL1: Q?.3 (D)
- new net SDA: Q?.1 (S), R?.2, U?.12 (SDA)
- new net SDA1: Q?.6 (D)
