File: kicad/DAC.sch (KiCad schematic (older format))
At the start: 32 parts

Commit message: update all passive footprints
Parts:
- C12, C13, C14, C15, C16, C17, C18, C19, C20, C21, C22, C23: renamed from C?; footprint Capacitor_SMD:C_0805_2012Metric -> Capacitor_SMD:C_0805_2012Metric_Pad1.18x1.45mm_HandSolder
- C24: renamed from C?; footprint Capacitor_SMD:C_0805_2012Metric_Pad1.15x1.40mm_HandSolder -> Capacitor_SMD:C_0805_2012Metric_Pad1.18x1.45mm_HandSolder
- R11, R12: renamed from R?; footprint Resistor_SMD:R_0805_2012Metric_Pad1.15x1.40mm_HandSolder -> Resistor_SMD:R_0805_2012Metric_Pad1.20x1.40mm_HandSolder
- R13, R14, R15, R16, R17, R18, R19, R20: renamed from R?; footprint Resistor_SMD:R_0805_2012Metric -> Resistor_SMD:R_0805_2012Metric_Pad1.20x1.40mm_HandSolder
- gave numbers to parts that had none: 4

Commit message: fixed usb5v-gnd bridge, continue placement
Parts:
- Q1: footprint (none) -> Package_TO_SOT_SMD:SOT-23-6_Handsoldering
Connections:
- net GND: no longer C12.1, C14.1, R11.1, R12.1, U6.3 (VIN), U7.14 (VCC)
- new net USB5V: C12.1, C14.1, R11.1, R12.1, U6.3 (VIN), U7.14 (VCC)
Changed lines of the file:
@@
 F 0 "Q1" V 4849 5600 50  0000 C CNN
 F 1 "Q_DUAL_NMOS_S1G1D2S2G2D1" V 4950 6100 50  0000 C CNN
-F 2 "" H 4800 5600 50  0001 C CNN
+F 2 "Package_TO_SOT_SMD:SOT-23-6_Handsoldering" H 4800 5600 50  0001 C CNN
 F 3 "~" H 4800 5600 50  0001 C CNN
 	1    4600 5600
@@
 F 0 "Q1" V 5299 5500 50  0000 C CNN
 F 1 "Q_DUAL_NMOS_S1G1D2S2G2D1" V 5400 6000 50  0000 C CNN
-F 2 "" H 5250 5500 50  0001 C CNN
+F 2 "Package_TO_SOT_SMD:SOT-23-6_Handsoldering" H 5250 5500 50  0001 C CNN
 F 3 "~" H 5250 5500 50  0001 C CNN
 	2    5050 5500
@@
 	4150 3500 4100 3500
 Wire Wire Line
-	4100 3500 4100 3650
-Wire Wire Line
 	4100 3650 4150 3650
 Text GLabel 4100 3400 0    50   Input ~ 0
@@
 Wire Wire Line
 	4100 3700 4100 3650
-Connection ~ 4100 3650
 $Comp
 L power:GND #PWR?

Commit message: more routing, add 2 new layers
Connections:
- net DAC2: now also U8.13 (-), U8.14; no longer U8.8, U8.9 (-)
- net DAC3: now also U8.8, U8.9 (-); no longer U8.13 (-), U8.14
- net at C22.2, R19.2: now also U8.12 (+); no longer U8.10 (+)
- net at C23.2, R20.2: now also U8.10 (+); no longer U8.12 (+)
Other:
- moved on the sheet: U8C, U8D
Changed lines of the file:
@@
 L Device:Opamp_Quad_Generic U?
 U 3 1 63AF84DB
-P 9450 4200
+P 9450 4700
 AR Path="/63AF84DB" Ref="U?"  Part="3"
 AR Path="/63922B28/63AF84DB" Ref="U8"  Part="3"
-F 0 "U8" H 9450 4200 50  0000 C CNN
-F 1 "TSV994IPT" H 9650 4350 50  0000 C CNN
-F 2 "Package_SO:TSSOP-14_4.4x5mm_P0.65mm" H 9450 4200 50  0001 C CNN
-F 3 "~" H 9450 4200 50  0001 C CNN
-	3    9450 4200
+F 0 "U8" H 9450 4700 50  0000 C CNN
+F 1 "TSV994IPT" H 9650 4850 50  0000 C CNN
+F 2 "Package_SO:TSSOP-14_4.4x5mm_P0.65mm" H 9450 4700 50  0001 C CNN
+F 3 "~" H 9450 4700 50  0001 C CNN
+	3    9450 4700
 	1    0    0    -1
 $EndComp
@@
 L Device:Opamp_Quad_Generic U?
 U 4 1 63AF84E1
-P 9450 4700
+P 9450 4200
 AR Path="/63AF84E1" Ref="U?"  Part="4"
 AR Path="/63922B28/63AF84E1" Ref="U8"  Part="4"
-F 0 "U8" H 9450 4700 50  0000 C CNN
-F 1 "TSV994IPT" H 9650 4850 50  0000 C CNN
-F 2 "Package_SO:TSSOP-14_4.4x5mm_P0.65mm" H 9450 4700 50  0001 C CNN
-F 3 "~" H 9450 4700 50  0001 C CNN
-	4    9450 4700
+F 0 "U8" H 9450 4200 50  0000 C CNN
+F 1 "TSV994IPT" H 9650 4350 50  0000 C CNN
+F 2 "Package_SO:TSSOP-14_4.4x5mm_P0.65mm" H 9450 4200 50  0001 C CNN
+F 3 "~" H 9450 4200 50  0001 C CNN
+	4    9450 4200
 	1    0    0    -1
 $EndComp

Commit message: finished route
Connections:
- net DAC0: now also U8.13 (-), U8.14; no longer U8.1, U8.2 (-)
- net DAC1: now also U8.8, U8.9 (-); no longer U8.6 (-), U8.7
- net DAC2: now also U8.1, U8.2 (-); no longer U8.13 (-), U8.14
- net DAC3: now also U8.6 (-), U8.7; no longer U8.8, U8.9 (-)
- net at C20.2, R17.2: now also U8.12 (+); no longer U8.3 (+)
- net at C21.2, R18.2: now also U8.10 (+); no longer U8.5 (+)
- net at C22.2, R19.2: now also U8.3 (+); no longer U8.12 (+)
- net at C23.2, R20.2: now also U8.5 (+); no longer U8.10 (+)
Other:
- moved on the sheet: U8A, U8B, U8C, U8D
Changed lines of the file:
@@
 L Device:Opamp_Quad_Generic U?
 U 1 1 63AF84CF
-P 9450 3250
+P 9450 4200
 AR Path="/63AF84CF" Ref="U?"  Part="1"
 AR Path="/63922B28/63AF84CF" Ref="U8"  Part="1"
+F 0 "U8" H 9450 4200 50  0000 C CNN
+F 1 "TSV994IPT" H 9650 3900 50  0000 C CNN
+F 2 "Package_SO:TSSOP-14_4.4x5mm_P0.65mm" H 9450 4200 50  0001 C CNN
+F 3 "~" H 9450 4200 50  0001 C CNN
+	1    9450 4200
+	1    0    0    -1
+$EndComp
+$Comp
+L Device:Opamp_Quad_Generic U?
+U 2 1 63AF84D5
+P 9450 4700
+AR Path="/63AF84D5" Ref="U?"  Part="2"
+AR Path="/63922B28/63AF84D5" Ref="U8"  Part="2"
+F 0 "U8" H 9450 4700 50  0000 C CNN
+F 1 "TSV994IPT" H 9650 5300 50  0000 C CNN
+F 2 "Package_SO:TSSOP-14_4.4x5mm_P0.65mm" H 9450 4700 50  0001 C CNN
+F 3 "~" H 9450 4700 50  0001 C CNN
+	2    9450 4700
+	1    0    0    -1
+$EndComp
+$Comp
+L Device:Opamp_Quad_Generic U?
+U 3 1 63AF84DB
+P 9450 3700
+AR Path="/63AF84DB" Ref="U?"  Part="3"
+AR Path="/63922B28/63AF84DB" Ref="U8"  Part="3"
+F 0 "U8" H 9450 3700 50  0000 C CNN
+F 1 "TSV994IPT" H 9650 3850 50  0000 C CNN
+F 2 "Package_SO:TSSOP-14_4.4x5mm_P0.65mm" H 9450 3700 50  0001 C CNN
+F 3 "~" H 9450 3700 50  0001 C CNN
+	3    9450 3700
+	1    0    0    -1
+$EndComp
+$Comp
+L Device:Opamp_Quad_Generic U?
+U 4 1 63AF84E1
+P 9450 3250
+AR Path="/63AF84E1" Ref="U?"  Part="4"
+AR Path="/63922B28/63AF84E1" Ref="U8"  Part="4"
 F 0 "U8" H 9450 3250 50  0000 C CNN
-F 1 "TSV994IPT" H 9650 2950 50  0000 C CNN
+F 1 "TSV994IPT" H 9650 3400 50  0000 C CNN
 F 2 "Package_SO:TSSOP-14_4.4x5mm_P0.65mm" H 9450 3250 50  0001 C CNN
 F 3 "~" H 9450 3250 50  0001 C CNN
-	1    9450 3250
-	1    0    0    -1
-$EndComp
-$Comp
-L Device:Opamp_Quad_Generic U?
-U 2 1 63AF84D5
-P 9450 3700
-AR Path="/63AF84D5" Ref="U?"  Part="2"
-AR Path="/63922B28/63AF84D5" Ref="U8"  Part="2"
-F 0 "U8" H 9450 3700 50  0000 C CNN
-F 1 "TSV994IPT" H 9650 4300 50  0000 C CNN
-F 2 "Package_SO:TSSOP-14_4.4x5mm_P0.65mm" H 9450 3700 50  0001 C CNN
-F 3 "~" H 9450 3700 50  0001 C CNN
-	2    9450 3700
-	1    0    0    -1
-$EndComp
-$Comp
-L Device:Opamp_Quad_Generic U?
-U 3 1 63AF84DB
-P 9450 4700
-AR Path="/63AF84DB" Ref="U?"  Part="3"
-AR Path="/63922B28/63AF84DB" Ref="U8"  Part="3"
-F 0 "U8" H 9450 4700 50  0000 C CNN
-F 1 "TSV994IPT" H 9650 4850 50  0000 C CNN
-F 2 "Package_SO:TSSOP-14_4.4x5mm_P0.65mm" H 9450 4700 50  0001 C CNN
-F 3 "~" H 9450 4700 50  0001 C CNN
-	3    9450 4700
-	1    0    0    -1
-$EndComp
-$Comp
-L Device:Opamp_Quad_Generic U?
-U 4 1 63AF84E1
-P 9450 4200
-AR Path="/63AF84E1" Ref="U?"  Part="4"
-AR Path="/63922B28/63AF84E1" Ref="U8"  Part="4"
-F 0 "U8" H 9450 4200 50  0000 C CNN
-F 1 "TSV994IPT" H 9650 4350 50  0000 C CNN
-F 2 "Package_SO:TSSOP-14_4.4x5mm_P0.65mm" H 9450 4200 50  0001 C CNN
-F 3 "~" H 9450 4200 50  0001 C CNN
-	4    9450 4200
+	4    9450 3250
 	1    0    0    -1
 $EndComp
@@
 	8800 3600 9150 3600
 Wire Wire Line
-	8800 4100 9150 4100
+	8800 4100 9100 4100
 Wire Wire Line
 	8800 4600 9150 4600
@@
 Wire Wire Line
 	1550 3700 1400 3700
+Connection ~ 9100 4100
+Wire Wire Line
+	9100 4100 9150 4100
 $EndSCHEMATC

Commit message: changing footprints
Parts:
- C12, C14, C15, C16, C17, C18, C19, C20, C21, C22, C23: value 0.1uF -> 0.1 uF; footprint Capacitor_SMD:C_0805_2012Metric_Pad1.18x1.45mm_HandSolder -> Capacitor_SMD:C_0603_1608Metric_Pad1.08x0.95mm_HandSolder
- C13, C24: value 1uF -> 1 uF
Changed lines of the file:
@@
 AR Path="/63922B28/63AF8404" Ref="C14"  Part="1"
 F 0 "C14" H 6950 3250 50  0000 L CNN
-F 1 "0.1uF" H 6850 3150 50  0000 L CNN
-F 2 "Capacitor_SMD:C_0805_2012Metric_Pad1.18x1.45mm_HandSolder" H 7150 3200 50  0001 C CNN
+F 1 "0.1 uF" H 6850 3150 50  0000 L CNN
+F 2 "Capacitor_SMD:C_0603_1608Metric_Pad1.08x0.95mm_HandSolder" H 7150 3200 50  0001 C CNN
 F 3 "~" H 7150 3200 50  0001 C CNN
 	1    7150 3200
@@
 AR Path="/63922B28/63AF8413" Ref="C15"  Part="1"
 F 0 "C15" H 6950 3650 50  0000 L CNN
-F 1 "0.1uF" H 6850 3550 50  0000 L CNN
-F 2 "Capacitor_SMD:C_0805_2012Metric_Pad1.18x1.45mm_HandSolder" H 7150 3600 50  0001 C CNN
+F 1 "0.1 uF" H 6850 3550 50  0000 L CNN
+F 2 "Capacitor_SMD:C_0603_1608Metric_Pad1.08x0.95mm_HandSolder" H 7150 3600 50  0001 C CNN
 F 3 "~" H 7150 3600 50  0001 C CNN
 	1    7150 3600
@@
 AR Path="/63922B28/63AF8433" Ref="C16"  Part="1"
 F 0 "C16" H 8600 3250 50  0000 L CNN
-F 1 "0.1uF" H 8600 3300 50  0000 L CNN
-F 2 "Capacitor_SMD:C_0805_2012Metric_Pad1.18x1.45mm_HandSolder" H 8500 3250 50  0001 C CNN
+F 1 "0.1 uF" H 8600 3300 50  0000 L CNN
+F 2 "Capacitor_SMD:C_0603_1608Metric_Pad1.08x0.95mm_HandSolder" H 8500 3250 50  0001 C CNN
 F 3 "~" H 8500 3250 50  0001 C CNN
 	1    8500 3250
@@
 AR Path="/63922B28/63AF8439" Ref="C20"  Part="1"
 F 0 "C20" H 8600 3300 50  0000 L CNN
-F 1 "0.1uF" H 8500 3400 50  0000 L CNN
-F 2 "Capacitor_SMD:C_0805_2012Metric_Pad1.18x1.45mm_HandSolder" H 8800 3250 50  0001 C CNN
+F 1 "0.1 uF" H 8500 3400 50  0000 L CNN
+F 2 "Capacitor_SMD:C_0603_1608Metric_Pad1.08x0.95mm_HandSolder" H 8800 3250 50  0001 C CNN
 F 3 "~" H 8800 3250 50  0001 C CNN
 	1    8800 3250
@@
 AR Path="/63922B28/63AF8459" Ref="C17"  Part="1"
 F 0 "C17" H 8600 3700 50  0000 L CNN
-F 1 "0.1uF" H 8600 3750 50  0000 L CNN
-F 2 "Capacitor_SMD:C_0805_2012Metric_Pad1.18x1.45mm_HandSolder" H 8500 3700 50  0001 C CNN
+F 1 "0.1 uF" H 8600 3750 50  0000 L CNN
+F 2 "Capacitor_SMD:C_0603_1608Metric_Pad1.08x0.95mm_HandSolder" H 8500 3700 50  0001 C CNN
 F 3 "~" H 8500 3700 50  0001 C CNN
 	1    8500 3700
@@
 AR Path="/63922B28/63AF845F" Ref="C21"  Part="1"
 F 0 "C21" H 8600 3750 50  0000 L CNN
-F 1 "0.1uF" H 8500 3850 50  0000 L CNN
-F 2 "Capacitor_SMD:C_0805_2012Metric_Pad1.18x1.45mm_HandSolder" H 8800 3700 50  0001 C CNN
+F 1 "0.1 uF" H 8500 3850 50  0000 L CNN
+F 2 "Capacitor_SMD:C_0603_1608Metric_Pad1.08x0.95mm_HandSolder" H 8800 3700 50  0001 C CNN
 F 3 "~" H 8800 3700 50  0001 C CNN
 	1    8800 3700
@@
 AR Path="/63922B28/63AF847F" Ref="C18"  Part="1"
 F 0 "C18" H 8600 4200 50  0000 L CNN
-F 1 "0.1uF" H 8600 4250 50  0000 L CNN
-F 2 "Capacitor_SMD:C_0805_2012Metric_Pad1.18x1.45mm_HandSolder" H 8500 4200 50  0001 C CNN
+F 1 "0.1 uF" H 8600 4250 50  0000 L CNN
+F 2 "Capacitor_SMD:C_0603_1608Metric_Pad1.08x0.95mm_HandSolder" H 8500 4200 50  0001 C CNN
 F 3 "~" H 8500 4200 50  0001 C CNN
 	1    8500 4200
@@
 AR Path="/63922B28/63AF8485" Ref="C22"  Part="1"
 F 0 "C22" H 8600 4250 50  0000 L CNN
-F 1 "0.1uF" H 8500 4350 50  0000 L CNN
-F 2 "Capacitor_SMD:C_0805_2012Metric_Pad1.18x1.45mm_HandSolder" H 8800 4200 50  0001 C CNN
+F 1 "0.1 uF" H 8500 4350 50  0000 L CNN
+F 2 "Capacitor_SMD:C_0603_1608Metric_Pad1.08x0.95mm_HandSolder" H 8800 4200 50  0001 C CNN
 F 3 "~" H 8800 4200 50  0001 C CNN
 	1    8800 4200
@@
 AR Path="/63922B28/63AF84AB" Ref="C23"  Part="1"
 F 0 "C23" H 8600 4700 50  0000 L CNN
-F 1 "0.1uF" H 8550 4800 50  0000 L CNN
-F 2 "Capacitor_SMD:C_0805_2012Metric_Pad1.18x1.45mm_HandSolder" H 8800 4700 50  0001 C CNN
+F 1 "0.1 uF" H 8550 4800 50  0000 L CNN
+F 2 "Capacitor_SMD:C_0603_1608Metric_Pad1.08x0.95mm_HandSolder" H 8800 4700 50  0001 C CNN
 F 3 "~" H 8800 4700 50  0001 C CNN
 	1    8800 4700
@@
 AR Path="/63922B28/63AF8501" Ref="C24"  Part="1"
 F 0 "C24" H 9465 5396 50  0000 L CNN
-F 1 "1uF" H 9465 5305 50  0000 L CNN
+F 1 "1 uF" H 9465 5305 50  0000 L CNN
 F 2 "Capacitor_SMD:C_0805_2012Metric_Pad1.18x1.45mm_HandSolder" H 9388 5200 50  0001 C CNN
 F 3 "~" H 9350 5350 50  0001 C CNN
@@
 	8800 3600 9150 3600
 Wire Wire Line
-	8800 4100 9100 4100
-Wire Wire Line
 	8800 4600 9150 4600
 $Comp
@@
 AR Path="/63922B28/63AF8554" Ref="C12"  Part="1"
 F 0 "C12" H 3700 3650 50  0000 L CNN
-F 1 "0.1uF" H 3600 3550 50  0000 L CNN
-F 2 "Capacitor_SMD:C_0805_2012Metric_Pad1.18x1.45mm_HandSolder" H 3900 3600 50  0001 C CNN
+F 1 "0.1 uF" H 3600 3550 50  0000 L CNN
+F 2 "Capacitor_SMD:C_0603_1608Metric_Pad1.08x0.95mm_HandSolder" H 3900 3600 50  0001 C CNN
 F 3 "~" H 3900 3600 50  0001 C CNN
 	1    3900 3600
@@
 AR Path="/63922B28/63AF855A" Ref="C13"  Part="1"
 F 0 "C13" H 5200 3600 50  0000 L CNN
-F 1 "1uF" H 5150 3500 50  0000 L CNN
+F 1 "1 uF" H 5150 3500 50  0000 L CNN
 F 2 "Capacitor_SMD:C_0805_2012Metric_Pad1.18x1.45mm_HandSolder" H 5100 3600 50  0001 C CNN
 F 3 "~" H 5100 3600 50  0001 C CNN
@@
 AR Path="/63922B28/63AF84A5" Ref="C19"  Part="1"
 F 0 "C19" H 8600 4700 50  0000 L CNN
-F 1 "0.1uF" H 8600 4750 50  0000 L CNN
-F 2 "Capacitor_SMD:C_0805_2012Metric_Pad1.18x1.45mm_HandSolder" H 8500 4700 50  0001 C CNN
+F 1 "0.1 uF" H 8600 4750 50  0000 L CNN
+F 2 "Capacitor_SMD:C_0603_1608Metric_Pad1.08x0.95mm_HandSolder" H 8500 4700 50  0001 C CNN
 F 3 "~" H 8500 4700 50  0001 C CNN
 	1    8500 4700
@@
 Wire Wire Line
 	1550 3700 1400 3700
-Connection ~ 9100 4100
-Wire Wire Line
-	9100 4100 9150 4100
+Wire Wire Line
+	8800 4100 9150 4100
 $EndSCHEMATC

Commit message: 0603 most passives
Parts:
- R11, R12, R13, R14, R15, R16, R17, R18, R19, R20: footprint Resistor_SMD:R_0805_2012Metric_Pad1.20x1.40mm_HandSolder -> Resistor_SMD:R_0603_1608Metric_Pad0.98x0.95mm_HandSolder
Changed lines of the file:
@@
 F 0 "R13" V 8250 3100 50  0000 L CNN
 F 1 "1k" V 8350 3100 50  0000 L CNN
-F 2 "Resistor_SMD:R_0805_2012Metric_Pad1.20x1.40mm_HandSolder" V 8280 3150 50  0001 C CNN
+F 2 "Resistor_SMD:R_0603_1608Metric_Pad0.98x0.95mm_HandSolder" V 8280 3150 50  0001 C CNN
 F 3 "~" H 8350 3150 50  0001 C CNN
 	1    8350 3150
@@
 F 0 "R17" V 8550 3100 50  0000 L CNN
 F 1 "1k" V 8650 3100 50  0000 L CNN
-F 2 "Resistor_SMD:R_0805_2012Metric_Pad1.20x1.40mm_HandSolder" V 8580 3150 50  0001 C CNN
+F 2 "Resistor_SMD:R_0603_1608Metric_Pad0.98x0.95mm_HandSolder" V 8580 3150 50  0001 C CNN
 F 3 "~" H 8650 3150 50  0001 C CNN
 	1    8650 3150
@@
 F 0 "R14" V 8250 3550 50  0000 L CNN
 F 1 "1k" V 8350 3550 50  0000 L CNN
-F 2 "Resistor_SMD:R_0805_2012Metric_Pad1.20x1.40mm_HandSolder" V 8280 3600 50  0001 C CNN
+F 2 "Resistor_SMD:R_0603_1608Metric_Pad0.98x0.95mm_HandSolder" V 8280 3600 50  0001 C CNN
 F 3 "~" H 8350 3600 50  0001 C CNN
 	1    8350 3600
@@
 F 0 "R18" V 8550 3550 50  0000 L CNN
 F 1 "1k" V 8650 3550 50  0000 L CNN
-F 2 "Resistor_SMD:R_0805_2012Metric_Pad1.20x1.40mm_HandSolder" V 8580 3600 50  0001 C CNN
+F 2 "Resistor_SMD:R_0603_1608Metric_Pad0.98x0.95mm_HandSolder" V 8580 3600 50  0001 C CNN
 F 3 "~" H 8650 3600 50  0001 C CNN
 	1    8650 3600
@@
 F 0 "R15" V 8250 4050 50  0000 L CNN
 F 1 "1k" V 8350 4050 50  0000 L CNN
-F 2 "Resistor_SMD:R_0805_2012Metric_Pad1.20x1.40mm_HandSolder" V 8280 4100 50  0001 C CNN
+F 2 "Resistor_SMD:R_0603_1608Metric_Pad0.98x0.95mm_HandSolder" V 8280 4100 50  0001 C CNN
 F 3 "~" H 8350 4100 50  0001 C CNN
 	1    8350 4100
@@
 F 0 "R19" V 8550 4050 50  0000 L CNN
 F 1 "1k" V 8650 4050 50  0000 L CNN
-F 2 "Resistor_SMD:R_0805_2012Metric_Pad1.20x1.40mm_HandSolder" V 8580 4100 50  0001 C CNN
+F 2 "Resistor_SMD:R_0603_1608Metric_Pad0.98x0.95mm_HandSolder" V 8580 4100 50  0001 C CNN
 F 3 "~" H 8650 4100 50  0001 C CNN
 	1    8650 4100
@@
 F 0 "R16" V 8250 4550 50  0000 L CNN
 F 1 "1k" V 8350 4550 50  0000 L CNN
-F 2 "Resistor_SMD:R_0805_2012Metric_Pad1.20x1.40mm_HandSolder" V 8280 4600 50  0001 C CNN
+F 2 "Resistor_SMD:R_0603_1608Metric_Pad0.98x0.95mm_HandSolder" V 8280 4600 50  0001 C CNN
 F 3 "~" H 8350 4600 50  0001 C CNN
 	1    8350 4600
@@
 F 0 "R20" V 8550 4550 50  0000 L CNN
 F 1 "1k" V 8650 4550 50  0000 L CNN
-F 2 "Resistor_SMD:R_0805_2012Metric_Pad1.20x1.40mm_HandSolder" V 8580 4600 50  0001 C CNN
+F 2 "Resistor_SMD:R_0603_1608Metric_Pad0.98x0.95mm_HandSolder" V 8580 4600 50  0001 C CNN
 F 3 "~" H 8650 4600 50  0001 C CNN
 	1    8650 4600
@@
 F 0 "R11" H 4170 5396 50  0000 L CNN
 F 1 "4.7k" H 4170 5305 50  0000 L CNN
-F 2 "Resistor_SMD:R_0805_2012Metric_Pad1.20x1.40mm_HandSolder" V 4030 5350 50  0001 C CNN
+F 2 "Resistor_SMD:R_0603_1608Metric_Pad0.98x0.95mm_HandSolder" V 4030 5350 50  0001 C CNN
 F 3 "~" H 4100 5350 50  0001 C CNN
 	1    4100 5350
@@
 F 0 "R12" H 4470 5396 50  0000 L CNN
 F 1 "4.7k" H 4470 5305 50  0000 L CNN
-F 2 "Resistor_SMD:R_0805_2012Metric_Pad1.20x1.40mm_HandSolder" V 4330 5350 50  0001 C CNN
+F 2 "Resistor_SMD:R_0603_1608Metric_Pad0.98x0.95mm_HandSolder" V 4330 5350 50  0001 C CNN
 F 3 "~" H 4400 5350 50  0001 C CNN
 	1    4400 5350

Commit message: adding jlc fields
Parts:
- C12, C14, C15, C16, C17, C18, C19, C20, C21, C22, C23: JLC (none) -> 0603; LCSC (none) -> C30926
- C13, C24: JLC (none) -> 0805; LCSC (none) -> C215803
- U6: JLC (none) -> SOT-23-5; LCSC (none) -> C698019
- U7: JLC (none) -> TDFN-14-EP(3x3); LCSC (none) -> C1554592
- U8: JLC (none) -> TSSOP-14; LCSC (none) -> C503311
Changed lines of the file:
@@
 F 2 "quadrant:SON40P300X500X80-15N" H 7900 3600 50  0001 C CNN
 F 3 "" H 7900 3600 50  0001 C CNN
+F 4 "TDFN-14-EP(3x3)" H 7900 3600 50  0001 C CNN "JLC"
+F 5 "C1554592" H 7900 3600 50  0001 C CNN "LCSC"
 	1    7900 3600
 	1    0    0    -1
@@
 F 2 "Capacitor_SMD:C_0603_1608Metric_Pad1.08x0.95mm_HandSolder" H 7150 3200 50  0001 C CNN
 F 3 "~" H 7150 3200 50  0001 C CNN
+F 4 "0603" H 7150 3200 50  0001 C CNN "JLC"
+F 5 "C30926" H 7150 3200 50  0001 C CNN "LCSC"
 	1    7150 3200
 	1    0    0    -1
@@
 F 2 "Capacitor_SMD:C_0603_1608Metric_Pad1.08x0.95mm_HandSolder" H 7150 3600 50  0001 C CNN
 F 3 "~" H 7150 3600 50  0001 C CNN
+F 4 "0603" H 7150 3600 50  0001 C CNN "JLC"
+F 5 "C30926" H 7150 3600 50  0001 C CNN "LCSC"
 	1    7150 3600
 	1    0    0    -1
@@
 F 2 "Capacitor_SMD:C_0603_1608Metric_Pad1.08x0.95mm_HandSolder" H 8500 3250 50  0001 C CNN
 F 3 "~" H 8500 3250 50  0001 C CNN
+F 4 "0603" H 8500 3250 50  0001 C CNN "JLC"
+F 5 "C30926" H 8500 3250 50  0001 C CNN "LCSC"
 	1    8500 3250
 	-1   0    0    1
@@
 F 2 "Capacitor_SMD:C_0603_1608Metric_Pad1.08x0.95mm_HandSolder" H 8800 3250 50  0001 C CNN
 F 3 "~" H 8800 3250 50  0001 C CNN
+F 4 "0603" H 8800 3250 50  0001 C CNN "JLC"
+F 5 "C30926" H 8800 3250 50  0001 C CNN "LCSC"
 	1    8800 3250
 	-1   0    0    1
@@
 F 2 "Capacitor_SMD:C_0603_1608Metric_Pad1.08x0.95mm_HandSolder" H 8500 3700 50  0001 C CNN
 F 3 "~" H 8500 3700 50  0001 C CNN
+F 4 "0603" H 8500 3700 50  0001 C CNN "JLC"
+F 5 "C30926" H 8500 3700 50  0001 C CNN "LCSC"
 	1    8500 3700
 	-1   0    0    1
@@
 F 2 "Capacitor_SMD:C_0603_1608Metric_Pad1.08x0.95mm_HandSolder" H 8800 3700 50  0001 C CNN
 F 3 "~" H 8800 3700 50  0001 C CNN
+F 4 "0603" H 8800 3700 50  0001 C CNN "JLC"
+F 5 "C30926" H 8800 3700 50  0001 C CNN "LCSC"
 	1    8800 3700
 	-1   0    0    1
@@
 F 2 "Capacitor_SMD:C_0603_1608Metric_Pad1.08x0.95mm_HandSolder" H 8500 4200 50  0001 C CNN
 F 3 "~" H 8500 4200 50  0001 C CNN
+F 4 "0603" H 8500 4200 50  0001 C CNN "JLC"
+F 5 "C30926" H 8500 4200 50  0001 C CNN "LCSC"
 	1    8500 4200
 	-1   0    0    1
@@
 F 2 "Capacitor_SMD:C_0603_1608Metric_Pad1.08x0.95mm_HandSolder" H 8800 4200 50  0001 C CNN
 F 3 "~" H 8800 4200 50  0001 C CNN
+F 4 "0603" H 8800 4200 50  0001 C CNN "JLC"
+F 5 "C30926" H 8800 4200 50  0001 C CNN "LCSC"
 	1    8800 4200
 	-1   0    0    1
@@
 F 2 "Capacitor_SMD:C_0603_1608Metric_Pad1.08x0.95mm_HandSolder" H 8800 4700 50  0001 C CNN
 F 3 "~" H 8800 4700 50  0001 C CNN
+F 4 "0603" H 8800 4700 50  0001 C CNN "JLC"
+F 5 "C30926" H 8800 4700 50  0001 C CNN "LCSC"
 	1    8800 4700
 	-1   0    0    1
@@
 F 2 "Package_SO:TSSOP-14_4.4x5mm_P0.65mm" H 9450 4200 50  0001 C CNN
 F 3 "~" H 9450 4200 50  0001 C CNN
+F 4 "TSSOP-14" H 9450 4200 50  0001 C CNN "JLC"
+F 5 "C503311" H 9450 4200 50  0001 C CNN "LCSC"
 	1    9450 4200
 	1    0    0    -1
@@
 F 2 "Package_SO:TSSOP-14_4.4x5mm_P0.65mm" H 9450 4700 50  0001 C CNN
 F 3 "~" H 9450 4700 50  0001 C CNN
+F 4 "TSSOP-14" H 9450 4700 50  0001 C CNN "JLC"
+F 5 "C503311" H 9450 4700 50  0001 C CNN "LCSC"
 	2    9450 4700
 	1    0    0    -1
@@
 F 2 "Package_SO:TSSOP-14_4.4x5mm_P0.65mm" H 9450 3700 50  0001 C CNN
 F 3 "~" H 9450 3700 50  0001 C CNN
+F 4 "TSSOP-14" H 9450 3700 50  0001 C CNN "JLC"
+F 5 "C503311" H 9450 3700 50  0001 C CNN "LCSC"
 	3    9450 3700
 	1    0    0    -1
@@
 F 2 "Package_SO:TSSOP-14_4.4x5mm_P0.65mm" H 9450 3250 50  0001 C CNN
 F 3 "~" H 9450 3250 50  0001 C CNN
+F 4 "TSSOP-14" H 9450 3250 50  0001 C CNN "JLC"
+F 5 "C503311" H 9450 3250 50  0001 C CNN "LCSC"
 	4    9450 3250
 	1    0    0    -1
@@
 F 2 "Package_SO:TSSOP-14_4.4x5mm_P0.65mm" H 9750 5350 50  0001 C CNN
 F 3 "~" H 9750 5350 50  0001 C CNN
+F 4 "TSSOP-14" H 9750 5350 50  0001 C CNN "JLC"
+F 5 "C503311" H 9750 5350 50  0001 C CNN "LCSC"
 	5    9750 5350
 	1    0    0    -1
@@
 F 2 "Capacitor_SMD:C_0805_2012Metric_Pad1.18x1.45mm_HandSolder" H 9388 5200 50  0001 C CNN
 F 3 "~" H 9350 5350 50  0001 C CNN
+F 4 "0805" H 9350 5350 50  0001 C CNN "JLC"
+F 5 "C215803" H 9350 5350 50  0001 C CNN "LCSC"
 	1    9350 5350
 	1    0    0    -1
@@
 F 3 "" H 4550 3550 50  0001 C CNN
 F 4 "https://www.digikey.com/en/products/detail/toshiba-semiconductor-and-storage/TCR2EE48-LM/5114341" H 4550 3550 50  0001 C CNN "digikey"
+F 5 "SOT-23-5" H 4550 3550 50  0001 C CNN "JLC"
+F 6 "C698019" H 4550 3550 50  0001 C CNN "LCSC"
 	1    4550 3550
 	1    0    0    -1
@@
 F 2 "Capacitor_SMD:C_0603_1608Metric_Pad1.08x0.95mm_HandSolder" H 3900 3600 50  0001 C CNN
 F 3 "~" H 3900 3600 50  0001 C CNN
+F 4 "0603" H 3900 3600 50  0001 C CNN "JLC"
+F 5 "C30926" H 3900 3600 50  0001 C CNN "LCSC"
 	1    3900 3600
 	1    0    0    -1
@@
 F 2 "Capacitor_SMD:C_0805_2012Metric_Pad1.18x1.45mm_HandSolder" H 5100 3600 50  0001 C CNN
 F 3 "~" H 5100 3600 50  0001 C CNN
+F 4 "0805" H 5100 3600 50  0001 C CNN "JLC"
+F 5 "C215803" H 5100 3600 50  0001 C CNN "LCSC"
 	1    5100 3600
 	1    0    0    -1
@@
 F 2 "Capacitor_SMD:C_0603_1608Metric_Pad1.08x0.95mm_HandSolder" H 8500 4700 50  0001 C CNN
 F 3 "~" H 8500 4700 50  0001 C CNN
+F 4 "0603" H 8500 4700 50  0001 C CNN "JLC"
+F 5 "C30926" H 8500 4700 50  0001 C CNN "LCSC"
 	1    8500 4700
 	-1   0    0    1
