File: kicad/DAC.sch (KiCad schematic (older format))
At the start: 27 parts, among them Q1 Q_DUAL_NMOS_S1G1D2S2G2D1, U6 TCR2EE48, U7 DS3911, U8 TSV994IPT

Commit message: more jlc fields
Parts:
- C12, C13, C14, C15, C16, C17, C18, C19, C20, C21, C22, C23, C24, U7, U8: ordered (none) -> y
- R11, R12: JLC (none) -> 0603; LCSC (none) -> C23162; ordered (none) -> y
- R13, R14, R15, R16, R17, R18, R19, R20: JLC (none) -> 0603; LCSC (none) -> C21190; ordered (none) -> y
- U6: value TCR2EE48 -> VRH4801NTX; ordered (none) -> ---
Changed lines of the file:
@@
 F 4 "TDFN-14-EP(3x3)" H 7900 3600 50  0001 C CNN "JLC"
 F 5 "C1554592" H 7900 3600 50  0001 C CNN "LCSC"
+F 6 "y" H 7900 3600 50  0001 C CNN "ordered"
 	1    7900 3600
 	1    0    0    -1
@@
 F 4 "0603" H 7150 3200 50  0001 C CNN "JLC"
 F 5 "C30926" H 7150 3200 50  0001 C CNN "LCSC"
+F 6 "y" H 7150 3200 50  0001 C CNN "ordered"
 	1    7150 3200
 	1    0    0    -1
@@
 F 4 "0603" H 7150 3600 50  0001 C CNN "JLC"
 F 5 "C30926" H 7150 3600 50  0001 C CNN "LCSC"
+F 6 "y" H 7150 3600 50  0001 C CNN "ordered"
 	1    7150 3600
 	1    0    0    -1
@@
 F 2 "Resistor_SMD:R_0603_1608Metric_Pad0.98x0.95mm_HandSolder" V 8280 3150 50  0001 C CNN
 F 3 "~" H 8350 3150 50  0001 C CNN
+F 4 "0603" H 8350 3150 50  0001 C CNN "JLC"
+F 5 " C21190 " H 8350 3150 50  0001 C CNN "LCSC"
+F 6 "y" H 8350 3150 50  0001 C CNN "ordered"
 	1    8350 3150
 	0    -1   1    0
@@
 F 4 "0603" H 8500 3250 50  0001 C CNN "JLC"
 F 5 "C30926" H 8500 3250 50  0001 C CNN "LCSC"
+F 6 "y" H 8500 3250 50  0001 C CNN "ordered"
 	1    8500 3250
 	-1   0    0    1
@@
 F 4 "0603" H 8800 3250 50  0001 C CNN "JLC"
 F 5 "C30926" H 8800 3250 50  0001 C CNN "LCSC"
+F 6 "y" H 8800 3250 50  0001 C CNN "ordered"
 	1    8800 3250
 	-1   0    0    1
@@
 F 2 "Resistor_SMD:R_0603_1608Metric_Pad0.98x0.95mm_HandSolder" V 8580 3150 50  0001 C CNN
 F 3 "~" H 8650 3150 50  0001 C CNN
+F 4 "0603" H 8650 3150 50  0001 C CNN "JLC"
+F 5 " C21190 " H 8650 3150 50  0001 C CNN "LCSC"
+F 6 "y" H 8650 3150 50  0001 C CNN "ordered"
 	1    8650 3150
 	0    -1   1    0
@@
 F 2 "Resistor_SMD:R_0603_1608Metric_Pad0.98x0.95mm_HandSolder" V 8280 3600 50  0001 C CNN
 F 3 "~" H 8350 3600 50  0001 C CNN
+F 4 "0603" H 8350 3600 50  0001 C CNN "JLC"
+F 5 " C21190 " H 8350 3600 50  0001 C CNN "LCSC"
+F 6 "y" H 8350 3600 50  0001 C CNN "ordered"
 	1    8350 3600
 	0    -1   1    0
@@
 F 4 "0603" H 8500 3700 50  0001 C CNN "JLC"
 F 5 "C30926" H 8500 3700 50  0001 C CNN "LCSC"
+F 6 "y" H 8500 3700 50  0001 C CNN "ordered"
 	1    8500 3700
 	-1   0    0    1
@@
 F 4 "0603" H 8800 3700 50  0001 C CNN "JLC"
 F 5 "C30926" H 8800 3700 50  0001 C CNN "LCSC"
+F 6 "y" H 8800 3700 50  0001 C CNN "ordered"
 	1    8800 3700
 	-1   0    0    1
@@
 F 2 "Resistor_SMD:R_0603_1608Metric_Pad0.98x0.95mm_HandSolder" V 8580 3600 50  0001 C CNN
 F 3 "~" H 8650 3600 50  0001 C CNN
+F 4 "0603" H 8650 3600 50  0001 C CNN "JLC"
+F 5 " C21190 " H 8650 3600 50  0001 C CNN "LCSC"
+F 6 "y" H 8650 3600 50  0001 C CNN "ordered"
 	1    8650 3600
 	0    -1   1    0
@@
 F 2 "Resistor_SMD:R_0603_1608Metric_Pad0.98x0.95mm_HandSolder" V 8280 4100 50  0001 C CNN
 F 3 "~" H 8350 4100 50  0001 C CNN
+F 4 "0603" H 8350 4100 50  0001 C CNN "JLC"
+F 5 " C21190 " H 8350 4100 50  0001 C CNN "LCSC"
+F 6 "y" H 8350 4100 50  0001 C CNN "ordered"
 	1    8350 4100
 	0    -1   1    0
@@
 F 4 "0603" H 8500 4200 50  0001 C CNN "JLC"
 F 5 "C30926" H 8500 4200 50  0001 C CNN "LCSC"
+F 6 "y" H 8500 4200 50  0001 C CNN "ordered"
 	1    8500 4200
 	-1   0    0    1
@@
 F 4 "0603" H 8800 4200 50  0001 C CNN "JLC"
 F 5 "C30926" H 8800 4200 50  0001 C CNN "LCSC"
+F 6 "y" H 8800 4200 50  0001 C CNN "ordered"
 	1    8800 4200
 	-1   0    0    1
@@
 F 2 "Resistor_SMD:R_0603_1608Metric_Pad0.98x0.95mm_HandSolder" V 8580 4100 50  0001 C CNN
 F 3 "~" H 8650 4100 50  0001 C CNN
+F 4 "0603" H 8650 4100 50  0001 C CNN "JLC"
+F 5 " C21190 " H 8650 4100 50  0001 C CNN "LCSC"
+F 6 "y" H 8650 4100 50  0001 C CNN "ordered"
 	1    8650 4100
 	0    -1   1    0
@@
 F 2 "Resistor_SMD:R_0603_1608Metric_Pad0.98x0.95mm_HandSolder" V 8280 4600 50  0001 C CNN
 F 3 "~" H 8350 4600 50  0001 C CNN
+F 4 "0603" H 8350 4600 50  0001 C CNN "JLC"
+F 5 " C21190 " H 8350 4600 50  0001 C CNN "LCSC"
+F 6 "y" H 8350 4600 50  0001 C CNN "ordered"
 	1    8350 4600
 	0    -1   1    0
@@
 F 4 "0603" H 8800 4700 50  0001 C CNN "JLC"
 F 5 "C30926" H 8800 4700 50  0001 C CNN "LCSC"
+F 6 "y" H 8800 4700 50  0001 C CNN "ordered"
 	1    8800 4700
 	-1   0    0    1
@@
 F 2 "Resistor_SMD:R_0603_1608Metric_Pad0.98x0.95mm_HandSolder" V 8580 4600 50  0001 C CNN
 F 3 "~" H 8650 4600 50  0001 C CNN
+F 4 "0603" H 8650 4600 50  0001 C CNN "JLC"
+F 5 " C21190 " H 8650 4600 50  0001 C CNN "LCSC"
+F 6 "y" H 8650 4600 50  0001 C CNN "ordered"
 	1    8650 4600
 	0    -1   1    0
@@
 F 4 "TSSOP-14" H 9450 4200 50  0001 C CNN "JLC"
 F 5 "C503311" H 9450 4200 50  0001 C CNN "LCSC"
+F 6 "y" H 9450 4200 50  0001 C CNN "ordered"
 	1    9450 4200
 	1    0    0    -1
@@
 F 4 "TSSOP-14" H 9450 4700 50  0001 C CNN "JLC"
 F 5 "C503311" H 9450 4700 50  0001 C CNN "LCSC"
+F 6 "y" H 9450 4700 50  0001 C CNN "ordered"
 	2    9450 4700
 	1    0    0    -1
@@
 F 4 "TSSOP-14" H 9450 3700 50  0001 C CNN "JLC"
 F 5 "C503311" H 9450 3700 50  0001 C CNN "LCSC"
+F 6 "y" H 9450 3700 50  0001 C CNN "ordered"
 	3    9450 3700
 	1    0    0    -1
@@
 F 4 "TSSOP-14" H 9450 3250 50  0001 C CNN "JLC"
 F 5 "C503311" H 9450 3250 50  0001 C CNN "LCSC"
+F 6 "y" H 9450 3250 50  0001 C CNN "ordered"
 	4    9450 3250
 	1    0    0    -1
@@
 F 4 "TSSOP-14" H 9750 5350 50  0001 C CNN "JLC"
 F 5 "C503311" H 9750 5350 50  0001 C CNN "LCSC"
+F 6 "y" H 9750 5350 50  0001 C CNN "ordered"
 	5    9750 5350
 	1    0    0    -1
@@
 F 4 "0805" H 9350 5350 50  0001 C CNN "JLC"
 F 5 "C215803" H 9350 5350 50  0001 C CNN "LCSC"
+F 6 "y" H 9350 5350 50  0001 C CNN "ordered"
 	1    9350 5350
 	1    0    0    -1
@@
 F 2 "Resistor_SMD:R_0603_1608Metric_Pad0.98x0.95mm_HandSolder" V 4030 5350 50  0001 C CNN
 F 3 "~" H 4100 5350 50  0001 C CNN
+F 4 "0603" H 4100 5350 50  0001 C CNN "JLC"
+F 5 " C23162 " H 4100 5350 50  0001 C CNN "LCSC"
+F 6 "y" H 4100 5350 50  0001 C CNN "ordered"
 	1    4100 5350
 	-1   0    0    -1
@@
 F 2 "Resistor_SMD:R_0603_1608Metric_Pad0.98x0.95mm_HandSolder" V 4330 5350 50  0001 C CNN
 F 3 "~" H 4400 5350 50  0001 C CNN
+F 4 "0603" H 4400 5350 50  0001 C CNN "JLC"
+F 5 " C23162 " H 4400 5350 50  0001 C CNN "LCSC"
+F 6 "y" H 4400 5350 50  0001 C CNN "ordered"
 	1    4400 5350
 	-1   0    0    -1
@@
 AR Path="/63922B28/63AF8548" Ref="U6"  Part="1"
 F 0 "U6" H 4300 3750 50  0000 C CNN
-F 1 "TCR2EE48" H 4500 3350 50  0000 C CNN
+F 1 "VRH4801NTX" H 4500 3350 50  0000 C CNN
 F 2 "Package_TO_SOT_SMD:SOT-553" H 4550 3550 50  0001 C CNN
 F 3 "" H 4550 3550 50  0001 C CNN
@@
 F 5 "SOT-23-5" H 4550 3550 50  0001 C CNN "JLC"
 F 6 "C698019" H 4550 3550 50  0001 C CNN "LCSC"
+F 7 "---" H 4550 3550 50  0001 C CNN "ordered"
 	1    4550 3550
 	1    0    0    -1
@@
 F 4 "0603" H 3900 3600 50  0001 C CNN "JLC"
 F 5 "C30926" H 3900 3600 50  0001 C CNN "LCSC"
+F 6 "y" H 3900 3600 50  0001 C CNN "ordered"
 	1    3900 3600
 	1    0    0    -1
@@
 F 4 "0805" H 5100 3600 50  0001 C CNN "JLC"
 F 5 "C215803" H 5100 3600 50  0001 C CNN "LCSC"
+F 6 "y" H 5100 3600 50  0001 C CNN "ordered"
 	1    5100 3600
 	1    0    0    -1
@@
 F 4 "0603" H 8500 4700 50  0001 C CNN "JLC"
 F 5 "C30926" H 8500 4700 50  0001 C CNN "LCSC"
+F 6 "y" H 8500 4700 50  0001 C CNN "ordered"
 	1    8500 4700
 	-1   0    0    1
