File: kicad/_autosave-quadrant.kicad_pcb (KiCad board)
At the start: 4 copper layers, 53 x 73.5 mm, 82 parts, among them J1 USB_C_Receptacle_USB2.0, J7 Conn_01x06, Q2 NCE3400, SW1 SW_Push, U1 AD5317RBRUZ-RL7, U2 W25Q128JVS, U3 VRH4801NTX, U4 RT9193-33GB, U5 LP5907MFX-2.8_NOPB, U9 RP2040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

Commit message: more route
Parts:
- moved C34 0.79 mm to (34.2, -27.8)
Connections:
- net SDI renamed SCK
- U9 pad 31: LED1 -> GATE3
- U9 pad 32: EN1 -> GATE2
- U9 pad 34: unconnected-(U9-GPIO22-Pad34) -> LED1
- U9 pad 35: GATE3 -> EN1
- U9 pad 36: GATE2 -> unconnected-(U9-GPIO24-Pad36)
Routing:
- net EN1: track 0.00 -> 65.3 mm
- net LED1: track 4.91 -> 65.7 mm
- net unconnected-(U9-GPIO25-Pad37): track 8.02 -> 0.00 mm
- net GATE2: track 53.0 -> 57.7 mm
- net +3V3: track 55.2 -> 52.9 mm
- net GATE3: track 52.4 -> 54.0 mm
- net Net-(U9-VREG_VOUT): track 31.4 -> 30.7 mm
- net GND: track 92.3 -> 91.8 mm, vias 16 -> 21
