File: kicad/_autosave-quadrant.kicad_pcb (KiCad board)
At the start: 4 copper layers, 53 x 73.5 mm, 87 parts, among them J1 USB_C_Receptacle_USB2.0, J7 Conn_01x06, Q2 NCE3400, SW1 SW_Push, U1 AD5317RBRUZ-RL7, U2 W25Q128JVS, U3 VRH4801NTX, U4 RT9193-33GB, U5 LP5907MFX-2.8_NOPB, U6 LTV-352T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

Commit message: moved midii and midio
Parts:
- moved D8 59.9 mm to (14.6, -2.50)
- moved R11 59.1 mm to (11.2, -3.91), turned to 90 degrees
- moved R12 59.0 mm to (12.0, -15.2)
- moved U6 48.7 mm to (14.5, -9.00), turned to 90 degrees
- moved MIDI0 44.0 mm to (48.5, -9.00), turned to 0 degrees
- moved MIDII1 44.0 mm to (4.50, -9.00), turned to 180 degrees
- moved R21 40.6 mm to (47.2, -2.75), turned to 0 degrees
- moved R22 34.4 mm to (44.2, -15.5)
- moved Q2 34.3 mm to (48.2, -16.2), turned to 0 degrees
- moved R25 4.08 mm to (37.2, -10.7), turned to -90 degrees
- moved R27 2.08 mm to (35.8, -10.7), turned to -90 degrees
- moved C36 0.79 mm to (20.5, -27.2)
- moved C34 0.56 mm to (34.5, -27.2)
Connections:
- R12 pad 1: +3v3 -> +3V3
Routing:
- net GATE1: track 0.00 -> 90.7 mm, vias 0 -> 2
- net TOF1_GPIO: track 2.17 -> 72.7 mm, vias 0 -> 2
- net GATE0: track 58.7 -> 102.6 mm, vias 1 -> 2
- net TOF3_GPIO: track 2.21 -> 34.6 mm
- net TOF2_GPIO: track 60.4 -> 34.9 mm
- net MIDIO: track 23.6 -> 6.97 mm
- net TOF0_GPIO: track 10.1 -> 26.0 mm
- net Net-(D8-A): track 0.00 -> 14.1 mm
- net Net-(MIDII1-PadR): track 0.00 -> 12.5 mm
- net USB5V: track 67.2 -> 61.0 mm, vias 3 -> 2
- net Net-(D8-K): track 0.00 -> 5.89 mm
- net SDA0: track 186.8 -> 191.8 mm, vias 8 -> 9
- net GND: track 67.7 -> 72.3 mm
- net Net-(MIDI0-PadR): track 4.14 -> 0.00 mm
- net ~{LDAC}: track 0.00 -> 3.49 mm
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