File: kicad-7/quadrant.kicad_sch (KiCad schematic)
At the start: 10 parts, among them J1 USB_C_Receptacle_USB2.0, U4 RT9193-33GB, U5 LP5907MFX-2.8_NOPB

Commit message: moved component labels
Parts:
- C40: JLC 0805 -> 0603; LCSC C215803 -> C277528
- U5: footprint (none) -> Package_TO_SOT_SMD:SOT-23-5
Changed lines of the file:
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@@
       (effects (font (size 1.27 1.27)))
     )
-    (property "Footprint" "" (at 105.41 95.25 0)
+    (property "Footprint" "Package_TO_SOT_SMD:SOT-23-5" (at 105.41 95.25 0)
       (effects (font (size 1.27 1.27)) hide)
     )
@@
       (effects (font (size 1.27 1.27)) hide)
     )
-    (property "JLC" "0805" (at 52.07 102.87 0)
+    (property "JLC" "0603" (at 52.07 102.87 0)
       (effects (font (size 1.27 1.27)) hide)
     )
-    (property "LCSC" "C215803" (at 52.07 102.87 0)
+    (property "LCSC" "C277528 " (at 52.07 102.87 0)
       (effects (font (size 1.27 1.27)) hide)
     )
