File: kicad-7/DAC.kicad_sch (KiCad schematic)
At the start: 27 parts, among them Q1 DMN601DMK-7, U3 VRH4801NTX, U7 DS3911, U8 TSV994IPT

Commit message: removed lcsc properties from passives
Parts:
- C12, C14, C15, C16, C17, C18, C19, C20, C21, C22, C23: LCSC C30926 -> (none)
- C13, C24: LCSC C215803 -> (none)
- R11, R12: LCSC C23162 -> (none)
- R13, R14, R15, R16, R17, R18, R19, R20: LCSC C21190 -> (none)
Changed lines of the file:
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@@
       (effects (font (size 1.27 1.27)) hide)
     )
-    (property "LCSC" "C30926" (at 181.61 81.28 0)
+    (property "LCSC" "" (at 181.61 81.28 0)
       (effects (font (size 1.27 1.27)) hide)
     )
@@
       (effects (font (size 1.27 1.27)) hide)
     )
-    (property "LCSC" "C30926" (at 181.61 91.44 0)
+    (property "LCSC" "" (at 181.61 91.44 0)
       (effects (font (size 1.27 1.27)) hide)
     )
@@
       (effects (font (size 1.27 1.27)) hide)
     )
-    (property "LCSC" " C21190 " (at 212.09 80.01 0)
+    (property "LCSC" "" (at 212.09 80.01 0)
       (effects (font (size 1.27 1.27)) hide)
     )
@@
       (effects (font (size 1.27 1.27)) hide)
     )
-    (property "LCSC" "C30926" (at 215.9 82.55 0)
+    (property "LCSC" "" (at 215.9 82.55 0)
       (effects (font (size 1.27 1.27)) hide)
     )
@@
       (effects (font (size 1.27 1.27)) hide)
     )
-    (property "LCSC" "C30926" (at 223.52 82.55 0)
+    (property "LCSC" "" (at 223.52 82.55 0)
       (effects (font (size 1.27 1.27)) hide)
     )
@@
       (effects (font (size 1.27 1.27)) hide)
     )
-    (property "LCSC" " C21190 " (at 219.71 80.01 0)
+    (property "LCSC" "" (at 219.71 80.01 0)
       (effects (font (size 1.27 1.27)) hide)
     )
@@
       (effects (font (size 1.27 1.27)) hide)
     )
-    (property "LCSC" " C21190 " (at 212.09 91.44 0)
+    (property "LCSC" "" (at 212.09 91.44 0)
       (effects (font (size 1.27 1.27)) hide)
     )
@@
       (effects (font (size 1.27 1.27)) hide)
     )
-    (property "LCSC" "C30926" (at 215.9 93.98 0)
+    (property "LCSC" "" (at 215.9 93.98 0)
       (effects (font (size 1.27 1.27)) hide)
     )
@@
       (effects (font (size 1.27 1.27)) hide)
     )
-    (property "LCSC" "C30926" (at 223.52 93.98 0)
+    (property "LCSC" "" (at 223.52 93.98 0)
       (effects (font (size 1.27 1.27)) hide)
     )
@@
       (effects (font (size 1.27 1.27)) hide)
     )
-    (property "LCSC" " C21190 " (at 219.71 91.44 0)
+    (property "LCSC" "" (at 219.71 91.44 0)
       (effects (font (size 1.27 1.27)) hide)
     )
@@
       (effects (font (size 1.27 1.27)) hide)
     )
-    (property "LCSC" " C21190 " (at 212.09 104.14 0)
+    (property "LCSC" "" (at 212.09 104.14 0)
       (effects (font (size 1.27 1.27)) hide)
     )
@@
       (effects (font (size 1.27 1.27)) hide)
     )
-    (property "LCSC" "C30926" (at 215.9 106.68 0)
+    (property "LCSC" "" (at 215.9 106.68 0)
       (effects (font (size 1.27 1.27)) hide)
     )
@@
       (effects (font (size 1.27 1.27)) hide)
     )
-    (property "LCSC" "C30926" (at 223.52 106.68 0)
+    (property "LCSC" "" (at 223.52 106.68 0)
       (effects (font (size 1.27 1.27)) hide)
     )
@@
       (effects (font (size 1.27 1.27)) hide)
     )
-    (property "LCSC" " C21190 " (at 219.71 104.14 0)
+    (property "LCSC" "" (at 219.71 104.14 0)
       (effects (font (size 1.27 1.27)) hide)
     )
@@
       (effects (font (size 1.27 1.27)) hide)
     )
-    (property "LCSC" " C21190 " (at 212.09 116.84 0)
+    (property "LCSC" "" (at 212.09 116.84 0)
       (effects (font (size 1.27 1.27)) hide)
     )
@@
       (effects (font (size 1.27 1.27)) hide)
     )
-    (property "LCSC" "C30926" (at 215.9 119.38 0)
+    (property "LCSC" "" (at 215.9 119.38 0)
       (effects (font (size 1.27 1.27)) hide)
     )
@@
       (effects (font (size 1.27 1.27)) hide)
     )
-    (property "LCSC" "C30926" (at 223.52 119.38 0)
+    (property "LCSC" "" (at 223.52 119.38 0)
       (effects (font (size 1.27 1.27)) hide)
     )
@@
       (effects (font (size 1.27 1.27)) hide)
     )
-    (property "LCSC" " C21190 " (at 219.71 116.84 0)
+    (property "LCSC" "" (at 219.71 116.84 0)
       (effects (font (size 1.27 1.27)) hide)
     )
@@
       (effects (font (size 1.27 1.27)) hide)
     )
-    (property "LCSC" "C215803" (at 237.49 135.89 0)
+    (property "LCSC" "" (at 237.49 135.89 0)
       (effects (font (size 1.27 1.27)) hide)
     )
@@
       (effects (font (size 1.27 1.27)) hide)
     )
-    (property "LCSC" " C23162 " (at 104.14 135.89 0)
+    (property "LCSC" "" (at 104.14 135.89 0)
       (effects (font (size 1.27 1.27)) hide)
     )
@@
       (effects (font (size 1.27 1.27)) hide)
     )
-    (property "LCSC" " C23162 " (at 111.76 135.89 0)
+    (property "LCSC" "" (at 111.76 135.89 0)
       (effects (font (size 1.27 1.27)) hide)
     )
@@
       (effects (font (size 1.27 1.27)) hide)
     )
-    (property "LCSC" "C30926" (at 99.06 91.44 0)
+    (property "LCSC" "" (at 99.06 91.44 0)
       (effects (font (size 1.27 1.27)) hide)
     )
@@
       (effects (font (size 1.27 1.27)) hide)
     )
-    (property "LCSC" "C215803" (at 129.54 91.44 0)
-      (effects (font (size 1.27 1.27)) hide)
-    )
+    (property "LCSC" "" (at 129.54 91.44 0)
+      (effects (font (size 1.27 1.27)) hide)
+    )
