File: kicad-7/mcu.kicad_sch (KiCad schematic)
At the start: 34 parts, among them J2 Conn_01x02_Male, J7 Conn_01x06, U2 W25Q128JVS, U9 RP2040, X1 XO53

Commit message: removed lcsc properties from passives
Parts:
- C27, C29, C30, C31, C32, C34, C35, C36, C37, C38: LCSC C30926 -> (none)
- C28, C33: LCSC C215803 -> (none)
- C39: LCSC C124567 -> (none)
- D0, D1, D2, D3: LCSC C84269 -> (none)
- R23, R24: LCSC C137753 -> (none)
- R25, R27: LCSC C22975 -> (none)
- R26, R28: LCSC C23162 -> (none)
- R29, R30, R31, R32: LCSC C109318 -> (none)
- R34: LCSC C21190 -> (none)
Changed lines of the file:
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@@
       (effects (font (size 1.27 1.27)) hide)
     )
-    (property "LCSC" "C30926" (at 76.2 62.23 0)
+    (property "LCSC" "" (at 76.2 62.23 0)
       (effects (font (size 1.27 1.27)) hide)
     )
@@
       (effects (font (size 1.27 1.27)) hide)
     )
-    (property "LCSC" " C21190 " (at 46.99 78.74 0)
+    (property "LCSC" "" (at 46.99 78.74 0)
       (effects (font (size 1.27 1.27)) hide)
     )
@@
       (effects (font (size 1.27 1.27)) hide)
     )
-    (property "LCSC" "C124567 " (at 63.5 111.76 0)
+    (property "LCSC" "" (at 63.5 111.76 0)
       (effects (font (size 1.27 1.27)) hide)
     )
@@
       (effects (font (size 1.27 1.27)) hide)
     )
-    (property "LCSC" "C22975" (at 191.77 77.47 0)
+    (property "LCSC" "" (at 191.77 77.47 0)
       (effects (font (size 1.27 1.27)) hide)
     )
@@
       (effects (font (size 1.27 1.27)) hide)
     )
-    (property "LCSC" "C22975" (at 184.15 77.47 0)
+    (property "LCSC" "" (at 184.15 77.47 0)
       (effects (font (size 1.27 1.27)) hide)
     )
@@
       (effects (font (size 1.27 1.27)) hide)
     )
-    (property "LCSC" "C84269" (at 204.47 106.68 0)
+    (property "LCSC" "" (at 204.47 106.68 0)
       (effects (font (size 1.27 1.27)) hide)
     )
@@
       (effects (font (size 1.27 1.27)) hide)
     )
-    (property "LCSC" "C109318 " (at 212.09 106.68 0)
+    (property "LCSC" "" (at 212.09 106.68 0)
       (effects (font (size 1.27 1.27)) hide)
     )
@@
       (effects (font (size 1.27 1.27)) hide)
     )
-    (property "LCSC" "C84269" (at 204.47 132.08 0)
+    (property "LCSC" "" (at 204.47 132.08 0)
       (effects (font (size 1.27 1.27)) hide)
     )
@@
       (effects (font (size 1.27 1.27)) hide)
     )
-    (property "LCSC" "C84269" (at 204.47 114.3 0)
+    (property "LCSC" "" (at 204.47 114.3 0)
       (effects (font (size 1.27 1.27)) hide)
     )
@@
       (effects (font (size 1.27 1.27)) hide)
     )
-    (property "LCSC" "C84269" (at 204.47 123.19 0)
+    (property "LCSC" "" (at 204.47 123.19 0)
       (effects (font (size 1.27 1.27)) hide)
     )
@@
       (effects (font (size 1.27 1.27)) hide)
     )
-    (property "LCSC" "C30926" (at 142.24 38.1 0)
+    (property "LCSC" "" (at 142.24 38.1 0)
       (effects (font (size 1.27 1.27)) hide)
     )
@@
       (effects (font (size 1.27 1.27)) hide)
     )
-    (property "LCSC" "C215803" (at 165.1 48.26 0)
+    (property "LCSC" "" (at 165.1 48.26 0)
       (effects (font (size 1.27 1.27)) hide)
     )
@@
       (effects (font (size 1.27 1.27)) hide)
     )
-    (property "LCSC" "C215803" (at 99.06 50.8 0)
+    (property "LCSC" "" (at 99.06 50.8 0)
       (effects (font (size 1.27 1.27)) hide)
     )
@@
       (effects (font (size 1.27 1.27)) hide)
     )
-    (property "LCSC" "C137753 " (at 170.18 63.5 0)
+    (property "LCSC" "" (at 170.18 63.5 0)
       (effects (font (size 1.27 1.27)) hide)
     )
@@
       (effects (font (size 1.27 1.27)) hide)
     )
-    (property "LCSC" "C137753 " (at 170.18 60.96 0)
+    (property "LCSC" "" (at 170.18 60.96 0)
       (effects (font (size 1.27 1.27)) hide)
     )
@@
       (effects (font (size 1.27 1.27)) hide)
     )
-    (property "LCSC" "C30926" (at 198.12 38.1 0)
+    (property "LCSC" "" (at 198.12 38.1 0)
       (effects (font (size 1.27 1.27)) hide)
     )
@@
       (effects (font (size 1.27 1.27)) hide)
     )
-    (property "LCSC" "C30926" (at 189.23 38.1 0)
+    (property "LCSC" "" (at 189.23 38.1 0)
       (effects (font (size 1.27 1.27)) hide)
     )
@@
       (effects (font (size 1.27 1.27)) hide)
     )
-    (property "LCSC" "C30926" (at 180.34 38.1 0)
+    (property "LCSC" "" (at 180.34 38.1 0)
       (effects (font (size 1.27 1.27)) hide)
     )
@@
       (effects (font (size 1.27 1.27)) hide)
     )
-    (property "LCSC" "C30926" (at 171.45 38.1 0)
+    (property "LCSC" "" (at 171.45 38.1 0)
       (effects (font (size 1.27 1.27)) hide)
     )
@@
       (effects (font (size 1.27 1.27)) hide)
     )
-    (property "LCSC" "C30926" (at 162.56 38.1 0)
+    (property "LCSC" "" (at 162.56 38.1 0)
       (effects (font (size 1.27 1.27)) hide)
     )
@@
       (effects (font (size 1.27 1.27)) hide)
     )
-    (property "LCSC" "C30926" (at 152.4 38.1 0)
+    (property "LCSC" "" (at 152.4 38.1 0)
       (effects (font (size 1.27 1.27)) hide)
     )
@@
       (effects (font (size 1.27 1.27)) hide)
     )
-    (property "LCSC" "C30926" (at 102.87 38.1 0)
+    (property "LCSC" "" (at 102.87 38.1 0)
       (effects (font (size 1.27 1.27)) hide)
     )
@@
       (effects (font (size 1.27 1.27)) hide)
     )
-    (property "LCSC" "C30926" (at 93.98 38.1 0)
+    (property "LCSC" "" (at 93.98 38.1 0)
       (effects (font (size 1.27 1.27)) hide)
     )
@@
       (effects (font (size 1.27 1.27)) hide)
     )
-    (property "LCSC" " C23162 " (at 191.77 93.98 0)
+    (property "LCSC" "" (at 191.77 93.98 0)
       (effects (font (size 1.27 1.27)) hide)
     )
@@
       (effects (font (size 1.27 1.27)) hide)
     )
-    (property "LCSC" " C23162 " (at 184.15 93.98 0)
+    (property "LCSC" "" (at 184.15 93.98 0)
       (effects (font (size 1.27 1.27)) hide)
     )
@@
       (effects (font (size 1.27 1.27)) hide)
     )
-    (property "LCSC" "C109318 " (at 212.09 114.3 0)
+    (property "LCSC" "" (at 212.09 114.3 0)
       (effects (font (size 1.27 1.27)) hide)
     )
@@
       (effects (font (size 1.27 1.27)) hide)
     )
-    (property "LCSC" "C109318 " (at 212.09 123.19 0)
+    (property "LCSC" "" (at 212.09 123.19 0)
       (effects (font (size 1.27 1.27)) hide)
     )
@@
       (effects (font (size 1.27 1.27)) hide)
     )
-    (property "LCSC" "C109318 " (at 212.09 132.08 0)
-      (effects (font (size 1.27 1.27)) hide)
-    )
+    (property "LCSC" "" (at 212.09 132.08 0)
+      (effects (font (size 1.27 1.27)) hide)
+    )

Commit message: replace reset jumper with switch
Parts:
- removed J2: Conn_01x02_Male, Connector_PinHeader_2.00mm:PinHeader_1x02_P2.00mm_Vertical, symbol quadrant-rescue:Conn_01x02_Male-Connector
- added SW1: SW_Push, Button_Switch_SMD:SW_Push_1P1T_NO_CK_KMR2, symbol Switch:SW_Push
Connections:
- net GND: now also SW1.1
- net at R34.2: now also SW1.2
Changed lines of the file:
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@@
     (stroke (width 0) (type default))
   )
-  (wire (pts (xy 43.18 81.28) (xy 43.18 86.36))
+  (wire (pts (xy 43.18 88.9) (xy 43.18 93.98))
     (stroke (width 0) (type default))
   )
@@
     )
   )
-  (symbol (lib_id "quadrant-rescue:Conn_01x02_Male-Connector") (at 38.1 78.74 0) (unit 1)
-    (in_bom yes) (on_board yes) (dnp no)
-    (property "Reference" "J2" (at 40.8432 74.1426 0)
-      (effects (font (size 1.27 1.27)))
-    )
-    (property "Value" "Conn_01x02_Male" (at 40.64 83.82 0)
-      (effects (font (size 1.27 1.27)))
-    )
-    (property "Footprint" "Connector_PinHeader_2.00mm:PinHeader_1x02_P2.00mm_Vertical" (at 38.1 78.74 0)
-      (effects (font (size 1.27 1.27)) hide)
-    )
-    (property "Datasheet" "~" (at 38.1 78.74 0)
-      (effects (font (size 1.27 1.27)) hide)
-    )
-    (property "JLC" "直插,P=2mm" (at 38.1 78.74 0)
-      (effects (font (size 1.27 1.27)) hide)
-    )
-    (property "LCSC" "C541856" (at 38.1 78.74 0)
-      (effects (font (size 1.27 1.27)) hide)
-    )
-    (property "ordered" "y" (at 38.1 78.74 0)
-      (effects (font (size 1.27 1.27)) hide)
-    )
-    (pin "1")
-    (pin "2")
-    (instances
-      (project "quadrant"
-        (path "/8946b391-7a1a-4938-822f-fe0b062d1674"
-          (reference "J2") (unit 1)
-        )
-        (path "/8946b391-7a1a-4938-822f-fe0b062d1674/00000000-0000-0000-0000-000063921d71"
-          (reference "J2") (unit 1)
-        )
-      )
-    )
-  )
-  (symbol (lib_id "power:GND") (at 43.18 86.36 0) (unit 1)
-    (in_bom yes) (on_board yes) (dnp no)
-    (property "Reference" "#PWR0104" (at 43.18 92.71 0)
-      (effects (font (size 1.27 1.27)) hide)
-    )
-    (property "Value" "GND" (at 43.307 90.7542 0)
-      (effects (font (size 1.27 1.27)))
-    )
-    (property "Footprint" "" (at 43.18 86.36 0)
-      (effects (font (size 1.27 1.27)) hide)
-    )
-    (property "Datasheet" "" (at 43.18 86.36 0)
+  (symbol (lib_id "power:GND") (at 43.18 93.98 0) (unit 1)
+    (in_bom yes) (on_board yes) (dnp no)
+    (property "Reference" "#PWR0104" (at 43.18 100.33 0)
+      (effects (font (size 1.27 1.27)) hide)
+    )
+    (property "Value" "GND" (at 43.307 98.3742 0)
+      (effects (font (size 1.27 1.27)))
+    )
+    (property "Footprint" "" (at 43.18 93.98 0)
+      (effects (font (size 1.27 1.27)) hide)
+    )
+    (property "Datasheet" "" (at 43.18 93.98 0)
       (effects (font (size 1.27 1.27)) hide)
     )
@@
         )
       )
+    )
+  )
+  (symbol (lib_id "Switch:SW_Push") (at 43.18 83.82 90) (unit 1)
+    (in_bom yes) (on_board yes) (dnp no) (fields_autoplaced)
+    (property "Reference" "SW1" (at 44.45 83.185 90)
+      (effects (font (size 1.27 1.27)) (justify right))
+    )
+    (property "Value" "SW_Push" (at 44.45 85.725 90)
+      (effects (font (size 1.27 1.27)) (justify right))
+    )
+    (property "Footprint" "Button_Switch_SMD:SW_Push_1P1T_NO_CK_KMR2" (at 38.1 83.82 0)
+      (effects (font (size 1.27 1.27)) hide)
+    )
+    (property "Datasheet" "~" (at 38.1 83.82 0)
+      (effects (font (size 1.27 1.27)) hide)
+    )
+    (pin "1")
+    (pin "2")
+    (instances
+      (project "quadrant"
+        (path "/8946b391-7a1a-4938-822f-fe0b062d1674/00000000-0000-0000-0000-000063921d71"
+          (reference "SW1") (unit 1)
+        )
+      )
